Commit message: Added geometry-aware ArUco navigation logic

File: src/warehouse_robot_bringup/urdf/gz_ros2_control.xacro (robot description, xacro)
@@ -1,32 +1,30 @@
 <?xml version="1.0"?>
-<!-- ros2_control hardware interface for Gazebo Harmonic (gz-sim).
-     Uses gz_ros2_control instead of gazebo_ros2_control.
-     Controls: diff drive wheels + fork prismatic joint. -->
 <robot xmlns:xacro="http://www.ros.org/wiki/xacro">
-    <ros2_control name="GzSimSystem" type="system">
+    <ros2_control name="GazeboSimSystem" type="system">
         <hardware>
             <plugin>gz_ros2_control/GazeboSimSystem</plugin>
         </hardware>
-        <!-- Drive wheels (velocity-controlled via DiffDriveController) -->
-        <joint name="right_wheel_joint">
-            <command_interface name="velocity"/>
+        <joint name="left_wheel_joint">
+            <command_interface name="velocity">
+                <param name="min">-10</param>
+                <param name="max">10</param>
+            </command_interface>
             <state_interface name="velocity"/>
             <state_interface name="position"/>
         </joint>
-        <joint name="left_wheel_joint">
-            <command_interface name="velocity"/>
+        <joint name="right_wheel_joint">
+            <command_interface name="velocity">
+                <param name="min">-10</param>
+                <param name="max">10</param>
+            </command_interface>
             <state_interface name="velocity"/>
             <state_interface name="position"/>
         </joint>
-        <!-- Fork prismatic joint (position-controlled for lift/lower) -->
         <joint name="fork_base_joint">
             <command_interface name="position"/>
-            <command_interface name="velocity"/>
             <state_interface name="position"/>
             <state_interface name="velocity"/>
-            <state_interface name="effort"/>
         </joint>
     </ros2_control>
-    <!-- gz_ros2_control plugin for Gazebo Harmonic -->
     <gazebo>
         <plugin filename="gz_ros2_control-system" name="gz_ros2_control::GazeboSimROS2ControlPlugin">

File: src/warehouse_robot_bringup/urdf/sensors.xacro (robot description, xacro)
@@ -32,7 +32,7 @@
     <!-- Gazebo Harmonic gpu_lidar sensor (publishes on gz-transport, bridged to /scan) -->
     <gazebo reference="laser_frame_link">
-        <sensor name="gpu_lidar" type="gpu_lidar">
+        <sensor name="lidar" type="lidar">
             <pose>0 0 0 0 0 0</pose>
-            <topic>lidar</topic>
+            <topic>/scan</topic>
             <update_rate>10</update_rate>
             <always_on>true</always_on>
@@ -47,10 +47,4 @@
                         <max_angle>3.14159</max_angle>
                     </horizontal>
-                    <vertical>
-                        <samples>1</samples>
-                        <resolution>1</resolution>
-                        <min_angle>0</min_angle>
-                        <max_angle>0</max_angle>
-                    </vertical>
                 </scan>
                 <range>
@@ -77,5 +71,5 @@
         <parent link="fork_base_link"/>
         <child link="camera_link"/>
-        <origin xyz="${fork_base_length / 2} 0 ${fork_base_height + 0.02}" rpy="0 0 0"/>
+        <origin xyz="${(fork_base_length / 2) + 0.05} 0 ${fork_base_height + 0.02}" rpy="0 0.5 0"/>
     </joint>
     <!-- Optical frame (standard ROS camera convention: Z-forward, X-right, Y-down) -->
@@ -94,5 +88,5 @@
             <always_on>true</always_on>
             <visualize>true</visualize>
-            <gz_frame_id>camera_link_optical</gz_frame_id>
+            <gz_frame_id>camera_link</gz_frame_id>
             <camera>
                 <horizontal_fov>1.089</horizontal_fov>

Commit message: Successfully added explore_lite source files

File: src/warehouse_robot_bringup/urdf/gz_ros2_control.xacro (robot description, xacro)
@@ -1,30 +1,32 @@
 <?xml version="1.0"?>
+<!-- ros2_control hardware interface for Gazebo Harmonic (gz-sim).
+     Uses gz_ros2_control instead of gazebo_ros2_control.
+     Controls: diff drive wheels + fork prismatic joint. -->
 <robot xmlns:xacro="http://www.ros.org/wiki/xacro">
-    <ros2_control name="GazeboSimSystem" type="system">
+    <ros2_control name="GzSimSystem" type="system">
         <hardware>
             <plugin>gz_ros2_control/GazeboSimSystem</plugin>
         </hardware>
-        <joint name="left_wheel_joint">
-            <command_interface name="velocity">
-                <param name="min">-10</param>
-                <param name="max">10</param>
-            </command_interface>
+        <!-- Drive wheels (velocity-controlled via DiffDriveController) -->
+        <joint name="right_wheel_joint">
+            <command_interface name="velocity"/>
             <state_interface name="velocity"/>
             <state_interface name="position"/>
         </joint>
-        <joint name="right_wheel_joint">
-            <command_interface name="velocity">
-                <param name="min">-10</param>
-                <param name="max">10</param>
-            </command_interface>
+        <joint name="left_wheel_joint">
+            <command_interface name="velocity"/>
             <state_interface name="velocity"/>
             <state_interface name="position"/>
         </joint>
+        <!-- Fork prismatic joint (position-controlled for lift/lower) -->
         <joint name="fork_base_joint">
             <command_interface name="position"/>
+            <command_interface name="velocity"/>
             <state_interface name="position"/>
             <state_interface name="velocity"/>
+            <state_interface name="effort"/>
         </joint>
     </ros2_control>
+    <!-- gz_ros2_control plugin for Gazebo Harmonic -->
     <gazebo>
         <plugin filename="gz_ros2_control-system" name="gz_ros2_control::GazeboSimROS2ControlPlugin">

File: src/warehouse_robot_bringup/urdf/sensors.xacro (robot description, xacro)
@@ -26,13 +26,20 @@
     </link>
     <joint name="laser_frame_joint" type="fixed">
+        <!-- Pallet-detection mount: low and forward.
+             Parent: chassis_bottom_link (origin sits at base_link z=0; ground is at z=-front_wheel_radius=-0.05).
+             X: 1.30 m places the laser between the lowered fork tines (gap y=-0.425..0.425) and ahead of the
+                lift_base front face at x=1.195 — so it does NOT live inside the mast/connector or chassis box.
+             Y: 0  (laterally centered between the forks).
+             Z: 0.15 m in chassis_bottom_link frame -> 0.20 m above the ground plane,
+                comfortably above the 0.076 m fork-tine tops and below the lift_body_connector top (0.505). -->
         <parent link="chassis_bottom_link"/>
         <child link="laser_frame_link"/>
-        <origin xyz="0 0 ${chassis_bottom_height + chassis_top_height + (laser_frame_length / 2)}" rpy="0 0 0" />
+        <origin xyz="1.30 0 0.15" rpy="0 0 0" />
     </joint>
     <!-- Gazebo Harmonic gpu_lidar sensor (publishes on gz-transport, bridged to /scan) -->
     <gazebo reference="laser_frame_link">
-        <sensor name="lidar" type="lidar">
+        <sensor name="gpu_lidar" type="gpu_lidar">
             <pose>0 0 0 0 0 0</pose>
-            <topic>/scan</topic>
+            <topic>lidar</topic>
             <update_rate>10</update_rate>
             <always_on>true</always_on>
@@ -47,7 +54,13 @@
                         <max_angle>3.14159</max_angle>
                     </horizontal>
+                    <vertical>
+                        <samples>1</samples>
+                        <resolution>1</resolution>
+                        <min_angle>0</min_angle>
+                        <max_angle>0</max_angle>
+                    </vertical>
                 </scan>
                 <range>
-                    <min>0.3</min>
+                    <min>0.08</min>
                     <max>12.0</max>
                     <resolution>0.01</resolution>
@@ -71,5 +84,5 @@
         <parent link="fork_base_link"/>
         <child link="camera_link"/>
-        <origin xyz="${(fork_base_length / 2) + 0.05} 0 ${fork_base_height + 0.02}" rpy="0 0.5 0"/>
+        <origin xyz="${fork_base_length / 2} 0 ${fork_base_height + 0.02}" rpy="0 0 0"/>
     </joint>
     <!-- Optical frame (standard ROS camera convention: Z-forward, X-right, Y-down) -->
@@ -88,5 +101,5 @@
             <always_on>true</always_on>
             <visualize>true</visualize>
-            <gz_frame_id>camera_link</gz_frame_id>
+            <gz_frame_id>camera_link_optical</gz_frame_id>
             <camera>
                 <horizontal_fov>1.089</horizontal_fov>
